File: TLA_InputOutput/Purrtico_TLA/Purrtico_TLA.kicad_sch (KiCad schematic)
At the start: 60 parts, among them J1 XLR3, J2 Conn_01x03, J3 Conn_01x02, J4 XLR3, J5 Conn_01x02, U1 OPA1679, U2 OPA1679

Commit message: added mounting holes
Parts:
- added H1, H2, H3, H4: MountingHole, MountingHole:MountingHole_3.2mm_M3_DIN965, symbol Mechanical:MountingHole
