File: TLA_InputOutput/Purrtico_TLA/Purrtico_TLA.kicad_pcb (KiCad board)
At the start: 2 copper layers, 100 x 50 mm, 65 parts, among them J1 XLR3, J2 Conn_01x03, J3 Conn_01x02, J4 XLR3, J5 Conn_01x02, U1 OPA1679, U2 OPA1679

Commit message: update PCB to r01
Parts:
- moved RV2 3.56 mm to (112.3, 120.9)
- moved R26 1.27 mm to (110.7, 117.9)
Routing:
- net Net-(R2-Pad1): track 20.5 -> 23.2 mm, vias 0 -> 2
- net Net-(U2A-+): track 23.4 -> 26.0 mm, vias 0 -> 2
- net Net-(R26-Pad1): track 5.41 -> 3.07 mm
- net +15V: track 83.4 -> 82.0 mm, vias 3 -> 0
- net Net-(U2A--): track 30.8 -> 32.1 mm, vias 0 -> 2
- net -15V: track 82.7 -> 81.6 mm, vias 3 -> 0
Other:
- board text added: "greyboxaudio.com Purrtico TLA r01"
- board text removed: "greyboxaudio.com Purrtico TLA r00"
