File: Purrtico_TLA/Purrtico_TLA.kicad_sch (KiCad schematic)
At the start: 66 parts, among them J1 XLR3, J3 Conn_01x02, J4 XLR3, J5 Conn_01x02, J7 Conn_02x05_Odd_Even, U1 OPA1679, U2 OPA1679

Commit message: update pcb
Other:
- title: Purrtico TLA Input & Output -> Purrtico TLA
- moved on the sheet: R15, R5
Changed lines of the file:
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@@
 	(paper "A4")
 	(title_block
-		(title "Purrtico TLA Input & Output")
-		(date "2024-07-18")
+		(title "Purrtico TLA")
+		(date "2024-08-02")
 		(rev "01")
 		(company "Greybox Audio")
@@
 	(wire
 		(pts
-			(xy 210.82 90.17) (xy 229.87 90.17)
+			(xy 217.17 90.17) (xy 229.87 90.17)
 		)
 		(stroke
@@
 	(wire
 		(pts
-			(xy 198.12 143.51) (xy 204.47 143.51)
+			(xy 198.12 143.51) (xy 210.82 143.51)
 		)
 		(stroke
@@
 	(wire
 		(pts
-			(xy 212.09 143.51) (xy 229.87 143.51)
+			(xy 218.44 143.51) (xy 229.87 143.51)
 		)
 		(stroke
@@
 	(wire
 		(pts
-			(xy 198.12 90.17) (xy 203.2 90.17)
+			(xy 198.12 90.17) (xy 209.55 90.17)
 		)
 		(stroke
@@
 	(text "CMRR\nTrim"
 		(exclude_from_sim no)
-		(at 221.234 111.506 0)
+		(at 223.266 110.998 0)
 		(effects
 			(font
@@
 		(dnp no)
 		(property "Reference" "U1"
-			(at 162.56 144.78 0)
+			(at 162.56 129.286 0)
 			(effects
 				(font
@@
 		)
 		(property "Value" "OPA1679"
-			(at 162.56 142.24 0)
+			(at 162.56 126.746 0)
 			(effects
 				(font
@@
 		(dnp no)
 		(property "Reference" "U1"
-			(at 205.74 93.98 0)
+			(at 205.232 78.74 0)
 			(effects
 				(font
@@
 		)
 		(property "Value" "OPA1679"
-			(at 205.74 91.44 0)
+			(at 205.232 76.2 0)
 			(effects
 				(font
@@
 	(symbol
 		(lib_id "Device:R")
-		(at 208.28 143.51 90)
+		(at 214.63 143.51 90)
 		(mirror x)
 		(unit 1)
@@
 		(dnp no)
 		(property "Reference" "R15"
-			(at 208.28 149.86 90)
+			(at 214.63 149.86 90)
 			(effects
 				(font
@@
 		)
 		(property "Value" "3k3"
-			(at 208.28 147.32 90)
+			(at 214.63 147.32 90)
 			(effects
 				(font
@@
 		)
 		(property "Footprint" "Resistor_SMD:R_1206_3216Metric"
-			(at 208.28 141.732 90)
+			(at 214.63 141.732 90)
 			(effects
 				(font
@@
 		)
 		(property "Datasheet" "~"
-			(at 208.28 143.51 0)
+			(at 214.63 143.51 0)
 			(effects
 				(font
@@
 		)
 		(property "Description" ""
-			(at 208.28 143.51 0)
+			(at 214.63 143.51 0)
 			(effects
 				(font
@@
 		(dnp no)
 		(property "Reference" "U1"
-			(at 177.8 91.44 0)
+			(at 177.292 76.2 0)
 			(effects
 				(font
@@
 		)
 		(property "Value" "OPA1679"
-			(at 177.8 88.9 0)
+			(at 177.292 73.66 0)
 			(effects
 				(font
@@
 	(symbol
 		(lib_id "Device:R")
-		(at 207.01 90.17 90)
+		(at 213.36 90.17 90)
 		(mirror x)
 		(unit 1)
@@
 		(dnp no)
 		(property "Reference" "R5"
-			(at 207.01 96.52 90)
+			(at 213.36 96.52 90)
 			(effects
 				(font
@@
 		)
 		(property "Value" "3k3"
-			(at 207.01 93.98 90)
+			(at 213.36 93.98 90)
 			(effects
 				(font
@@
 		)
 		(property "Footprint" "Resistor_SMD:R_1206_3216Metric"
-			(at 207.01 88.392 90)
+			(at 213.36 88.392 90)
 			(effects
 				(font
@@
 		)
 		(property "Datasheet" "~"
-			(at 207.01 90.17 0)
+			(at 213.36 90.17 0)
 			(effects
 				(font
@@
 		)
 		(property "Description" ""
-			(at 207.01 90.17 0)
+			(at 213.36 90.17 0)
 			(effects
 				(font
@@
 		(dnp no)
 		(property "Reference" "U1"
-			(at 205.74 147.32 0)
+			(at 205.74 132.08 0)
 			(effects
 				(font
@@
 		)
 		(property "Value" "OPA1679"
-			(at 205.74 144.78 0)
+			(at 205.74 129.54 0)
 			(effects
 				(font
@@
 		(dnp no)
 		(property "Reference" "U2"
-			(at 97.79 57.15 0)
+			(at 97.536 42.164 0)
 			(effects
 				(font
@@
 		)
 		(property "Value" "OPA1679"
-			(at 97.79 54.61 0)
+			(at 97.536 39.624 0)
 			(effects
 				(font
@@
 		(dnp no)
 		(property "Reference" "U2"
-			(at 102.87 100.33 0)
+			(at 102.87 84.074 0)
 			(effects
 				(font
@@
 		)
 		(property "Value" "OPA1679"
-			(at 102.87 97.79 0)
+			(at 102.87 81.534 0)
 			(effects
 				(font
@@
 		(dnp no)
 		(property "Reference" "U2"
-			(at 163.83 167.64 0)
+			(at 163.83 172.466 0)
 			(effects
 				(font

Commit message: update circuit
Parts:
- removed RV3: 10k, Connector_PinHeader_2.54mm:PinHeader_1x03_P2.54mm_Vertical, symbol Device:R_Potentiometer
- added R33: 1k, Resistor_SMD:R_1206_3216Metric, symbol Device:R
- R19: value 1k -> 10k
- R7: value 2k2 -> 3k3
Connections:
- net at U1.10 (+): now also R19.2, R33.1
- net at R14.1, U1.9 (-): no longer R19.2
- net at C5.2: now also R33.2
Other:
- note added: "-3 dB 0°"
- note removed: "Output Trim"
- moved on the sheet: C5, J3, R19
