File: Purrtico_TLA/Purrtico_TLA.kicad_pcb (KiCad board)
At the start: 2 copper layers, 100 x 50 mm, 77 parts, among them J1 XLR3, J3 Conn_01x02, J4 XLR3, J5 Conn_01x02, J7 Conn_02x05_Odd_Even, U1 OPA1679, U2 OPA1679

Commit message: switch HPF knob
Parts:
- RV3: value 100k -> 100k log
- moved R26 1.78 mm to (93.2, 70.6)
Connections:
- RV3 pad 1: Net-(C21-Pad2) -> Net-(R34-Pad1)
- RV3 pad 2: Net-(R34-Pad1) -> Net-(C21-Pad2)
- RV3 pad 3: Net-(R34-Pad1) -> Net-(C21-Pad2)
- RV3 pad 4: Net-(U2D-+) -> Net-(R36-Pad2)
- RV3 pad 5: Net-(R36-Pad2) -> Net-(U2D-+)
- RV3 pad 6: Net-(R36-Pad2) -> Net-(U2D-+)
Routing:
- net Net-(C21-Pad2): track 16.6 -> 22.7 mm
- net Net-(R36-Pad2): track 4.63 -> 9.14 mm
- net Net-(U2D-+): track 20.2 -> 23.7 mm
- net GND: track 38.9 -> 36.9 mm
- net Net-(R26-Pad1): track 10.6 -> 11.7 mm
- net Net-(U2C-+): track 39.5 -> 38.9 mm

Commit message: added fabrication outputs
Connections:
- RV3 pad 1: Net-(R34-Pad1) -> Net-(C21-Pad2)
- RV3 pad 2: Net-(C21-Pad2) -> Net-(R34-Pad1)
- RV3 pad 3: Net-(C21-Pad2) -> Net-(R34-Pad1)
- RV3 pad 4: Net-(R36-Pad2) -> Net-(U2D-+)
- RV3 pad 5: Net-(U2D-+) -> Net-(R36-Pad2)
- RV3 pad 6: Net-(U2D-+) -> Net-(R36-Pad2)
Routing:
- net Net-(C21-Pad2): track 22.7 -> 16.6 mm
- net Net-(R36-Pad2): track 9.14 -> 4.89 mm
- net Net-(R34-Pad1): track 21.3 -> 25.6 mm
- net Net-(U2D-+): track 23.7 -> 20.8 mm

Commit message: moved rv3
Parts:
- moved RV3 0.51 mm to (89.5, 78.7)
Routing:
- net Net-(R36-Pad2): track 4.89 -> 6.09 mm
- net Net-(C21-Pad2): track 16.6 -> 16.0 mm
